File: mcu_sheet.kicad_sch (KiCad schematic)
At the start: 21 parts, among them J1 Conn_01x05, SW1 SW_Push, SW2 SW_SPDT, U1 STM32L4P5CETx, Y1 Crystal_GND23

Commit message: Comecei a adicionar a parte das entradas e continuo mexendo na parte do STM32
Parts:
- added D3: LED, BajaKICAD:LED_1210_HandSoldering, symbol Device:LED
- added R3: 1k, Resistor_SMD:R_1206_3216Metric_Pad1.30x1.75mm_HandSolder, symbol Device:R
Connections:
- net GND: now also D3.1 (K); no longer U1.23 (VSS), U1.35 (VSS), U1.47 (VSS), U1.8 (VSSA)
- new net: D3.2 (A), R3.2
- new net BD_LED: R3.1
- new net GNDA: U1.8 (VSSA)
- new net GNDD: U1.23 (VSS), U1.35 (VSS), U1.47 (VSS)
Other:
- note added: "LED Placa"
- note added: "Nota: Separa o GND analógico do digital, para evitar ruído"
- moved on the sheet: BT1, C1, C2, C3, C4, C5, C6, C7, C8, C9, D1, D2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
